Commit message: removed unneccessary meshes and modified mesh for ankle

File: src/mono/urdf/mono.urdf (robot description, URDF)
Before this commit: robot mono, 17 links, 16 joints
Joints:
- joint l_ankle_pitch_joint: limit lower=-2.8274333886 upper=2.8274333886 effort=10000 velocity=3 -> lower=-2.8274333886 upper=2.8274333886 effort=10 velocity=3
- joint l_ankle_roll_joint: limit lower=-2.8274333886 upper=2.8274333886 effort=10000 velocity=3 -> lower=-2.8274333886 upper=2.8274333886 effort=10 velocity=3
- joint l_hip_pitch_joint: limit lower=-2.8274333886 upper=2.8274333886 effort=10000 velocity=3 -> lower=-2.8274333886 upper=2.8274333886 effort=10 velocity=3
- joint l_hip_roll_joint: limit lower=-2.8274333886 upper=2.8274333886 effort=10000 velocity=3 -> lower=-2.8274333886 upper=2.8274333886 effort=10 velocity=3
- joint l_hip_yaw_joint: limit lower=-2.8274333886 upper=2.8274333886 effort=10000 velocity=3 -> lower=-2.8274333886 upper=2.8274333886 effort=10 velocity=3
- joint l_knee_pitch_joint: limit lower=-2.8274333886 upper=2.8274333886 effort=10000 velocity=3 -> lower=-2.8274333886 upper=2.8274333886 effort=10 velocity=3
- joint r_ankle_pitch_joint: limit lower=-2.8274333886 upper=2.8274333886 effort=10000 velocity=3 -> lower=-2.8274333886 upper=2.8274333886 effort=10 velocity=3
- joint r_ankle_roll_joint: limit lower=-2.8274333886 upper=2.8274333886 effort=10000 velocity=3 -> lower=-2.8274333886 upper=2.8274333886 effort=10 velocity=3
- joint r_hip_pitch_joint: limit lower=-2.8274333886 upper=2.8274333886 effort=10000 velocity=3 -> lower=-2.8274333886 upper=2.8274333886 effort=10 velocity=3
- joint r_hip_roll_joint: limit lower=-2.8274333886 upper=2.8274333886 effort=10000 velocity=3 -> lower=-2.8274333886 upper=2.8274333886 effort=10 velocity=3
- joint r_hip_yaw_joint: limit lower=-2.8274333886 upper=2.8274333886 effort=10000 velocity=3 -> lower=-2.8274333886 upper=2.8274333886 effort=10 velocity=3
- joint r_knee_pitch_joint: limit lower=-2.8274333886 upper=2.8274333886 effort=10000 velocity=3 -> lower=-2.8274333886 upper=2.8274333886 effort=10 velocity=3
