Commit message: added pybullet urdf

File: src/mono/urdf/Original Copy/2nd revision/mono.urdf (robot description, URDF)
Before this commit: robot mono, 17 links, 16 joints
Joints:
- joint l_ankle_pitch_joint: limit lower=-2.8274333886 upper=2.8274333886 effort=2 velocity=3 -> lower=-2.8274333886 upper=2.8274333886 effort=5 velocity=3
- joint l_ankle_roll_joint: limit lower=-2.8274333886 upper=2.8274333886 effort=2.5 velocity=3 -> lower=-2.8274333886 upper=2.8274333886 effort=3 velocity=3
- joint l_hip_pitch_joint: limit lower=-2.8274333886 upper=2.8274333886 effort=6 velocity=3 -> lower=-2.8274333886 upper=2.8274333886 effort=10 velocity=3
- joint l_hip_roll_joint: limit lower=-2.8274333886 upper=2.8274333886 effort=5 velocity=3 -> lower=-2.8274333886 upper=2.8274333886 effort=10 velocity=3
- joint l_hip_yaw_joint: limit lower=-2.8274333886 upper=2.8274333886 effort=5 velocity=3 -> lower=-2.8274333886 upper=2.8274333886 effort=10 velocity=3
- joint l_knee_pitch_joint: limit lower=-2.8274333886 upper=2.8274333886 effort=6 velocity=3 -> lower=-2.8274333886 upper=2.8274333886 effort=10 velocity=3
- joint r_ankle_pitch_joint: limit lower=-2.8274333886 upper=2.8274333886 effort=2 velocity=3 -> lower=-2.8274333886 upper=2.8274333886 effort=3 velocity=3
- joint r_ankle_roll_joint: limit lower=-2.8274333886 upper=2.8274333886 effort=2.5 velocity=3 -> lower=-2.8274333886 upper=2.8274333886 effort=3 velocity=3
- joint r_hip_pitch_joint: limit lower=-2.8274333886 upper=2.8274333886 effort=6 velocity=3 -> lower=-2.8274333886 upper=2.8274333886 effort=10 velocity=3
- joint r_hip_roll_joint: limit lower=-2.8274333886 upper=2.8274333886 effort=5 velocity=3 -> lower=-2.8274333886 upper=2.8274333886 effort=10 velocity=3
- joint r_hip_yaw_joint: limit lower=-2.8274333886 upper=2.8274333886 effort=5 velocity=3 -> lower=-2.8274333886 upper=2.8274333886 effort=10 velocity=3
- joint r_knee_pitch_joint: limit lower=-2.8274333886 upper=2.8274333886 effort=6 velocity=3 -> lower=-2.8274333886 upper=2.8274333886 effort=10 velocity=3

File: src/mono/urdf/Original Copy/3rd revision/mono.urdf (robot description, URDF)
Before this commit: robot mono, 17 links, 16 joints
Joints:
- joint l_ankle_pitch_joint: limit lower=-2.8274333886 upper=2.8274333886 effort=2 velocity=3 -> lower=-2.8274333886 upper=2.8274333886 effort=2.5 velocity=3
- joint l_hip_pitch_joint: limit lower=-2.8274333886 upper=2.8274333886 effort=6 velocity=3 -> lower=-2.8274333886 upper=2.8274333886 effort=10 velocity=3
- joint l_hip_roll_joint: limit lower=-2.8274333886 upper=2.8274333886 effort=5 velocity=3 -> lower=-2.8274333886 upper=2.8274333886 effort=10 velocity=3
- joint l_hip_yaw_joint: limit lower=-2.8274333886 upper=2.8274333886 effort=5 velocity=3 -> lower=-2.8274333886 upper=2.8274333886 effort=10 velocity=3
- joint l_knee_pitch_joint: limit lower=-2.8274333886 upper=2.8274333886 effort=6 velocity=3 -> lower=-2.8274333886 upper=2.8274333886 effort=10 velocity=3
- joint r_ankle_pitch_joint: limit lower=-2.8274333886 upper=2.8274333886 effort=2 velocity=3 -> lower=-2.8274333886 upper=2.8274333886 effort=2.5 velocity=3
- joint r_hip_pitch_joint: limit lower=-2.8274333886 upper=2.8274333886 effort=6 velocity=3 -> lower=-2.8274333886 upper=2.8274333886 effort=10 velocity=3
- joint r_hip_roll_joint: limit lower=-2.8274333886 upper=2.8274333886 effort=5 velocity=3 -> lower=-2.8274333886 upper=2.8274333886 effort=10 velocity=3
- joint r_hip_yaw_joint: limit lower=-2.8274333886 upper=2.8274333886 effort=5 velocity=3 -> lower=-2.8274333886 upper=2.8274333886 effort=10 velocity=3
- joint r_knee_pitch_joint: limit lower=-2.8274333886 upper=2.8274333886 effort=6 velocity=3 -> lower=-2.8274333886 upper=2.8274333886 effort=10 velocity=3

File: src/mono/urdf/mono_bullet.urdf (robot description, URDF)
Before this commit: robot mono, 17 links, 16 joints
Links:
- removed link base_link
- removed link imu_link
- removed link l_foot_ft_link
- removed link r_foot_ft_link
Joints:
- removed joint base_fixed
- removed joint imu_fixed
- removed joint l_ft_fixed
- removed joint r_ft_fixed
